File: schematic/stepper cape.brd (EAGLE design)
At the start: 87.3 x 55.9 mm, 49 parts, among them J1 ISP, U1 CAT24C, U2 LM7805, X1 A4988BREAKOUT

Commit message: Connected spare IO pins on AVR to inputs 0 and 1; changed to 0805 parts instead of 1206.
Parts:
- C3, C4: device adafruit:C1206 -> SparkFun-Passives:0805
- R1, R10, R11, R12, R13, R14, R15, R16, R17, R18, R2, R3, R4, R5, R6, R7, R8, R9: device adafruit:R1206 -> adafruit:R0805
Connections:
- net IN_0: now also U$2.4
- net IN_1: now also U$2.5
Routing:
- net IN_0: track 10.4 -> 50.6 mm, vias 0 -> 1
- net IN_1: track 17.8 -> 55.5 mm, vias 0 -> 1
- net GND: track 291.4 -> 294.5 mm
- net N$8: track 19.4 -> 17.9 mm
- net +3V3: track 164.1 -> 165.0 mm
- net N$22: track 26.4 -> 25.6 mm
- net N$7: track 16.3 -> 15.6 mm
